File: KiCad/GR_Color_Organ.kicad_pcb (KiCad board)
At the start: 2 copper layers, 46.9 x 41.4 mm, 55 parts, among them J1 Conn_01x03, J2 Conn_01x02, J3 Conn_01x02, J4 Conn_01x02, J5 Conn_01x02, J6 Conn_01x02, Q1 2N3904, Q2 2N3904, Q3 2N3904, Q4 2N3904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

Commit message: Add files via upload
Parts:
- removed C11, C4, C5, C8: 1uF, Capacitor_THT:C_Disc_D3.8mm_W2.6mm_P2.50mm
- removed Q3, Q5, Q7: 2N3904, Package_TO_SOT_THT:TO-92_Inline
- removed R10, R15, R20, R8: 1K, Resistor_THT:R_Axial_DIN0204_L3.6mm_D1.6mm_P2.54mm_Vertical
- removed R12, R17, R2, R9: 10K, Resistor_THT:R_Axial_DIN0204_L3.6mm_D1.6mm_P2.54mm_Vertical
- C10: value 100nF -> 1nF
- C3: value 100nF -> 220nF
- C6: value 2.2uF -> 15nF
- C7: value 100nF -> 33nF
- C9: value 2.2uF -> 1.5nF
- R3: value 100K -> 47K
- moved J2 12.3 mm to (121.0, 69.2)
- moved J4 12.3 mm to (121.1, 76.5)
- moved J5 12.3 mm to (121.2, 83.9)
- moved G*** 2.58 mm to (129.3, 75.7)
Connections:
- Q1 pad 1: Net-(C4-Pad1) -> GNDREF
- Q1 pad 3: Net-(Q1-Pad3) -> /Low_Out
- Q2 pad 1: Net-(C5-Pad1) -> GNDREF
- Q4 pad 1: Net-(C8-Pad1) -> GNDREF
- Q4 pad 3: Net-(Q4-Pad3) -> /Mid_Out
- Q6 pad 1: Net-(C11-Pad1) -> GNDREF
- Q6 pad 3: Net-(Q6-Pad3) -> /High_Out
- R3 pad 1: +5V -> Net-(Q2-Pad3)
Routing:
- net +5V: track 111.5 -> 90.9 mm
- net Net-(C8-Pad1): track 17.6 -> 0.00 mm
- net Net-(C11-Pad1): track 17.1 -> 0.00 mm
- net Net-(C4-Pad1): track 16.5 -> 0.00 mm
- net Net-(Q1-Pad3): track 10.5 -> 0.00 mm
- net Net-(Q4-Pad3): track 10.4 -> 0.00 mm
- net Net-(Q6-Pad3): track 10.0 -> 0.00 mm
- net Net-(C5-Pad1): track 8.55 -> 0.00 mm
- net Net-(Q2-Pad3): track 42.2 -> 46.8 mm
- net /Low_Out: track 12.7 -> 8.95 mm
- net /High_Out: track 15.8 -> 12.5 mm
- net /V+: track 62.8 -> 61.2 mm, vias 3 -> 2
- net /Mid_Out: track 12.2 -> 10.7 mm
Other:
- board text added: "A.In"
- board text removed: "Audio In"
